File: pcb/ocf4riser.sch (EAGLE design)
At the start: 39 parts, among them IC1 STM32F405RGTx, IC2 MCP1703CB, IC3 W25Q80BVSN, IC4 TPD3E001DRL, J1 TEENSY_3.1-3.2_DIL, J2 SWD/JTAG, J3 DEBUG, J4 IO, J5 I2C, J6 02X1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

Commit message: Tweaks
Parts:
- removed IC4: TPD3E001DRL, pld-usb-ti:TPD3E001DRL
- C2, C3: value 33p -> 27p
- L1: device EagleLibrary_Wuerth_Elektronik_eiSos_rev16a:WE-CBF_0603(HC) -> EagleLibrary_Wuerth_Elektronik_eiSos_rev16a:WE-CBF_0603(WB/HS)
Connections:
- net GND: no longer IC4.GND
- net USB_ID: no longer IC4.IO1
- net USB_I_N: no longer IC4.IO3
- net USB_I_P: no longer IC4.IO2
- net USB_VBUS: no longer IC4.VCC
Other:
- note added: "NOTE Most of the OTG functionality (e.g. power switching) offloaded to expansion. ESD protection also"
- note removed: "NOTE Most of the OTG functionality (e.g. power switching) offloaded to expansion."
- moved on the sheet: USBEX
Changed lines of the file:
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@@
 <part name="GND3" library="supply1" deviceset="GND" device=""/>
 <part name="X1" library="pld-txc" deviceset="TXC-7A" device=""/>
-<part name="C2" library="pld-rcl" deviceset="C-US" device="C0402" value="33p"/>
-<part name="C3" library="pld-rcl" deviceset="C-US" device="C0402" value="33p"/>
+<part name="C2" library="pld-rcl" deviceset="C-US" device="C0402" value="27p"/>
+<part name="C3" library="pld-rcl" deviceset="C-US" device="C0402" value="27p"/>
 <part name="GND4" library="supply1" deviceset="GND" device=""/>
 <part name="J2" library="pld-misc" deviceset="CORTEX_DEBUG" device="NAKED" value="SWD/JTAG"/>
@@
 <part name="C14" library="pld-rcl" deviceset="C-US" device="C0603" value="1u"/>
 <part name="GND12" library="supply1" deviceset="GND" device=""/>
-<part name="L1" library="EagleLibrary_Wuerth_Elektronik_eiSos_rev16a" deviceset="WE-CBF" device="_0603(HC)"/>
-<part name="IC4" library="pld-usb-ti" deviceset="TPD3E001" device="DRL"/>
-<part name="GND13" library="supply1" deviceset="GND" device=""/>
+<part name="L1" library="EagleLibrary_Wuerth_Elektronik_eiSos_rev16a" deviceset="WE-CBF" device="_0603(WB/HS)"/>
 <part name="R3" library="pld-rcl" deviceset="R-US_" device="R0402" value="22"/>
 <part name="R4" library="pld-rcl" deviceset="R-US_" device="R0402" value="22"/>
@@
 0 = system, 1 = SRAM</text>
 <text x="187.96" y="45.72" size="1.778" layer="97">WP + HOLD high</text>
-<text x="12.7" y="99.06" size="1.778" layer="97">NOTE
-Most of the OTG functionality (e.g.
-power switching) offloaded to expansion.</text>
+<text x="12.7" y="83.82" size="1.778" layer="97">NOTE
+Most of the OTG functionality (e.g. power
+switching) offloaded to expansion. ESD
+protection also</text>
 <text x="261.62" y="119.38" size="1.778" layer="97">Crystal Cl=18p
 C = 2x(Cl - Cp)
@@
 <instance part="GND12" gate="1" x="233.68" y="111.76"/>
 <instance part="L1" gate="G$1" x="210.82" y="129.54"/>
-<instance part="IC4" gate="G$1" x="63.5" y="58.42"/>
-<instance part="GND13" gate="1" x="76.2" y="48.26"/>
 <instance part="R3" gate="G$1" x="38.1" y="30.48"/>
 <instance part="R4" gate="G$1" x="30.48" y="35.56"/>
@@
 <instance part="C17" gate="G$1" x="86.36" y="226.06"/>
 <instance part="GND23" gate="1" x="86.36" y="213.36"/>
-<instance part="+3V14" gate="G$1" x="78.74" y="93.98" rot="MR0"/>
-<instance part="GND24" gate="1" x="78.74" y="68.58"/>
-<instance part="USBEX" gate="G$1" x="93.98" y="83.82"/>
+<instance part="+3V14" gate="G$1" x="78.74" y="78.74" rot="MR0"/>
+<instance part="GND24" gate="1" x="78.74" y="53.34"/>
+<instance part="USBEX" gate="G$1" x="93.98" y="68.58"/>
 <instance part="J7" gate="G$1" x="93.98" y="33.02"/>
 </instances>
@@
 </segment>
 <segment>
-<wire x1="83.82" y1="86.36" x2="78.74" y2="86.36" width="0.1524" layer="91"/>
+<wire x1="83.82" y1="71.12" x2="78.74" y2="71.12" width="0.1524" layer="91"/>
 <pinref part="+3V14" gate="G$1" pin="+3V3"/>
-<wire x1="78.74" y1="91.44" x2="78.74" y2="86.36" width="0.1524" layer="91"/>
+<wire x1="78.74" y1="76.2" x2="78.74" y2="71.12" width="0.1524" layer="91"/>
 <pinref part="USBEX" gate="G$1" pin="1"/>
 </segment>
@@
 </segment>
 <segment>
-<pinref part="IC4" gate="G$1" pin="GND"/>
-<wire x1="73.66" y1="55.88" x2="76.2" y2="55.88" width="0.1524" layer="91"/>
-<pinref part="GND13" gate="1" pin="GND"/>
-<wire x1="76.2" y1="55.88" x2="76.2" y2="50.8" width="0.1524" layer="91"/>
-</segment>
-<segment>
 <wire x1="355.6" y1="68.58" x2="353.06" y2="68.58" width="0.1524" layer="91"/>
 <wire x1="353.06" y1="68.58" x2="353.06" y2="66.04" width="0.1524" layer="91"/>
@@
 </segment>
 <segment>
-<wire x1="83.82" y1="76.2" x2="78.74" y2="76.2" width="0.1524" layer="91"/>
+<wire x1="83.82" y1="60.96" x2="78.74" y2="60.96" width="0.1524" layer="91"/>
 <pinref part="GND24" gate="1" pin="GND"/>
-<wire x1="78.74" y1="76.2" x2="78.74" y2="71.12" width="0.1524" layer="91"/>
+<wire x1="78.74" y1="60.96" x2="78.74" y2="55.88" width="0.1524" layer="91"/>
 <pinref part="USBEX" gate="G$1" pin="5"/>
 </segment>
@@
 <wire x1="83.82" y1="35.56" x2="81.28" y2="35.56" width="0.1524" layer="91"/>
 <wire x1="81.28" y1="35.56" x2="81.28" y2="45.72" width="0.1524" layer="91"/>
-<pinref part="IC4" gate="G$1" pin="VCC"/>
-<wire x1="81.28" y1="45.72" x2="81.28" y2="60.96" width="0.1524" layer="91"/>
-<wire x1="81.28" y1="60.96" x2="73.66" y2="60.96" width="0.1524" layer="91"/>
 <wire x1="116.84" y1="45.72" x2="81.28" y2="45.72" width="0.1524" layer="91"/>
 <junction x="116.84" y="45.72"/>
-<junction x="81.28" y="45.72"/>
 <pinref part="J7" gate="G$1" pin="1"/>
 </segment>
@@
 <segment>
 <pinref part="USBEX" gate="G$1" pin="4"/>
-<label x="22.86" y="25.4" size="1.778" layer="95" rot="R180"/>
-<pinref part="IC4" gate="G$1" pin="IO1"/>
-<wire x1="45.72" y1="25.4" x2="22.86" y2="25.4" width="0.1524" layer="91"/>
-<wire x1="53.34" y1="60.96" x2="45.72" y2="60.96" width="0.1524" layer="91"/>
-<wire x1="45.72" y1="60.96" x2="45.72" y2="25.4" width="0.1524" layer="91"/>
-<wire x1="83.82" y1="78.74" x2="45.72" y2="78.74" width="0.1524" layer="91"/>
-<wire x1="45.72" y1="78.74" x2="45.72" y2="60.96" width="0.1524" layer="91"/>
-<junction x="45.72" y="60.96"/>
+<label x="81.28" y="63.5" size="1.778" layer="95" rot="R180"/>
+<wire x1="83.82" y1="63.5" x2="81.28" y2="63.5" width="0.1524" layer="91"/>
 </segment>
 </net>
@@
 <wire x1="83.82" y1="33.02" x2="73.66" y2="33.02" width="0.1524" layer="91"/>
 <wire x1="73.66" y1="33.02" x2="73.66" y2="35.56" width="0.1524" layer="91"/>
-<wire x1="73.66" y1="35.56" x2="50.8" y2="35.56" width="0.1524" layer="91"/>
+<wire x1="73.66" y1="35.56" x2="35.56" y2="35.56" width="0.1524" layer="91"/>
 <pinref part="R4" gate="G$1" pin="2"/>
-<pinref part="IC4" gate="G$1" pin="IO3"/>
-<wire x1="50.8" y1="35.56" x2="35.56" y2="35.56" width="0.1524" layer="91"/>
-<wire x1="50.8" y1="55.88" x2="53.34" y2="55.88" width="0.1524" layer="91"/>
-<wire x1="50.8" y1="55.88" x2="50.8" y2="35.56" width="0.1524" layer="91"/>
-<junction x="50.8" y="35.56"/>
 <pinref part="J7" gate="G$1" pin="2"/>
 </segment>
@@
 <net name="USB_I_P" class="1">
 <segment>
-<wire x1="83.82" y1="30.48" x2="48.26" y2="30.48" width="0.1524" layer="91"/>
+<wire x1="83.82" y1="30.48" x2="43.18" y2="30.48" width="0.1524" layer="91"/>
 <pinref part="R3" gate="G$1" pin="2"/>
-<pinref part="IC4" gate="G$1" pin="IO2"/>
-<wire x1="48.26" y1="30.48" x2="43.18" y2="30.48" width="0.1524" layer="91"/>
-<wire x1="53.34" y1="58.42" x2="48.26" y2="58.42" width="0.1524" layer="91"/>
-<wire x1="48.26" y1="58.42" x2="48.26" y2="30.48" width="0.1524" layer="91"/>
-<junction x="48.26" y="30.48"/>
 <pinref part="J7" gate="G$1" pin="3"/>
 </segment>
@@
 <segment>
 <pinref part="USBEX" gate="G$1" pin="3"/>
-<wire x1="81.28" y1="81.28" x2="83.82" y2="81.28" width="0.1524" layer="91"/>
-<label x="81.28" y="81.28" size="1.778" layer="95" rot="R180"/>
+<wire x1="81.28" y1="66.04" x2="83.82" y2="66.04" width="0.1524" layer="91"/>
+<label x="81.28" y="66.04" size="1.778" layer="95" rot="R180"/>
 </segment>
 </net>
@@
 <segment>
 <pinref part="USBEX" gate="G$1" pin="2"/>
-<wire x1="81.28" y1="83.82" x2="83.82" y2="83.82" width="0.1524" layer="91"/>
-<label x="81.28" y="83.82" size="1.778" layer="95" rot="R180"/>
-</segment>
-</net>
+<wire x1="81.28" y1="68.58" x2="83.82" y2="68.58" width="0.1524" layer="91"/>
+<label x="81.28" y="68.58" size="1.778" layer="95" rot="R180"/>
+</segment>
+</net>
